File: project.kicad_pcb (KiCad board)
At the start: 4 copper layers, 88.8 x 70.1 mm, 69 parts, among them J1 USB3_B, J2 Jumper_3_Open, J3 Jumper_3_Open, J4 Jumper_3_Open, J6 Conn_02x10_Odd_Even, SW1 SW_Push, U1 CYUSB3014, U2 Conn_02x32_Odd_Even, U3 M25P80, U4 MP2359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

Commit message: everything routed
Parts:
- moved C25 189.2 mm to (186.9, 78.3)
- moved C13 188.5 mm to (166.1, 109.7)
- moved C17 188.5 mm to (172.8, 105.1)
- moved C23 188.5 mm to (138.6, 82.7)
- moved C5 188.5 mm to (166.6, 112.0)
- moved J1 188.5 mm to (156.3, 83.3)
- moved R13 188.5 mm to (139.3, 100.0)
- moved R16 188.5 mm to (132.1, 84.3)
- moved R21 188.5 mm to (167.4, 126.4)
- moved R8 188.5 mm to (179.1, 102.1)
- moved U1 188.5 mm to (157.6, 107.5)
- moved C1 188.5 mm to (156.7, 98.0)
- moved C10 188.5 mm to (149.8, 110.2)
- moved C11 188.5 mm to (162.7, 116.9)
- moved C12 188.5 mm to (167.3, 104.8)
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Connections:
- U1 pad C4: I2C-MCLK -> I2S-MCLK
Routing:
- net +1V2: track 35.2 -> 150.4 mm, vias 29 -> 32
- net VBUS_5V: track 4.79 -> 119.5 mm, vias 20 -> 21
- net TCK: track 0.78 -> 49.1 mm
- net CTRL5: track 0.45 -> 45.7 mm
- net D1: track 0.45 -> 45.7 mm
- net CTRL6: track 0.49 -> 45.6 mm
- net D30: track 0.49 -> 45.5 mm
- net D5: track 0.49 -> 45.5 mm
- net CTRL4: track 0.49 -> 45.5 mm
- net CTRL8: track 0.45 -> 45.5 mm
- net CTRL3: track 0.35 -> 45.4 mm
- net D23: track 0.38 -> 45.4 mm
- net D14: track 0.45 -> 45.5 mm
- net D24: track 0.42 -> 45.4 mm
- net D7: track 0.49 -> 45.5 mm
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- added copper zone on PWR, net +3V3
- added copper zone on B.Cu, net Earth
- added copper zone on B.Cu, net VBUS_5V
- added copper zone on PWR, net VBUS_5V
- removed copper zone on PWR, net +1V2
- removed copper zone on B.Cu, net +3V3
Other:
- net class Default: clearance 0.13 -> 0.1
- rule trace_clearance: 0.13 -> 0.1
