File: project.kicad_pcb (KiCad board)
At the start: 4 copper layers, 88.8 x 70.1 mm, 69 parts, among them J1 USB3_B, J2 Jumper_3_Open, J3 Jumper_3_Open, J4 Jumper_3_Open, J6 Conn_02x10_Odd_Even, SW1 SW_Push, U1 CYUSB3014, U2 Conn_02x32_Odd_Even, U3 M25P80, U4 MP2359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

Commit message: 5v on pwr plane
Routing:
- net 5V_IN: track 13.2 -> 16.2 mm
Other:
- outline, holes or cut-outs redrawn
Changed lines of the file:
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@@
   (general
     (thickness 1.6)
-    (drawings 5)
-    (tracks 9098)
+    (drawings 9)
+    (tracks 9100)
     (zones 0)
     (modules 69)
@@
   (page A4)
   (layers
-    (0 F.Cu signal hide)
+    (0 F.Cu signal)
     (1 GND signal hide)
-    (2 PWR signal hide)
+    (2 PWR signal)
     (31 B.Cu signal hide)
     (32 B.Adhes user)
@@
   )
   (setup
-    (last_trace_width 0.75)
+    (last_trace_width 2)
     (user_trace_width 0.13)
     (user_trace_width 0.13)
@@
     )
   )
+  (gr_circle (center 196 127) (end 194 126) (layer Edge.Cuts) (width 0.05))
+  (gr_circle (center 119 127) (end 117 127) (layer Edge.Cuts) (width 0.05))
+  (gr_circle (center 196 73) (end 194 72) (layer Edge.Cuts) (width 0.05))
+  (gr_circle (center 119 73) (end 117 72) (layer Edge.Cuts) (width 0.05))
   (gr_line (start 113.2 68.36) (end 113.2 68.41) (layer Edge.Cuts) (width 0.05))
   (gr_line (start 202.03 68.36) (end 113.2 68.36) (layer Edge.Cuts) (width 0.05))
@@
   (segment (start 154.3905 99.821092) (end 155.7705 101.201092) (width 0.2286) (layer F.Cu) (net 82))
   (segment (start 196.92 132.47618) (end 197.03858 132.59476) (width 1) (layer F.Cu) (net 83))
-  (segment (start 197.03858 122.288589) (end 196.92 122.170009) (width 3) (layer PWR) (net 83))
-  (segment (start 197.03858 135.13476) (end 197.03858 122.288589) (width 3) (layer PWR) (net 83))
+  (segment (start 196.92 121.61) (end 200 124.69) (width 2) (layer PWR) (net 83))
+  (segment (start 200 129.63334) (end 197.03858 132.59476) (width 2) (layer PWR) (net 83))
+  (segment (start 200 124.69) (end 200 129.63334) (width 2) (layer PWR) (net 83))
+  (segment (start 197.03858 132.59476) (end 197.03858 135.13476) (width 2) (layer PWR) (net 83))
   (segment (start 158.8954 132.0646) (end 158.8954 132.55158) (width 0.13) (layer F.Cu) (net 84))
   (segment (start 158.902922 131.997843) (end 158.8954 132.0646) (width 0.13) (layer F.Cu) (net 84))

Commit message: added logo
Parts:
- added REF**: OSHW-Logo2_7.3x6mm_SilkScreen, Symbol:OSHW-Logo2_7.3x6mm_SilkScreen, F.Cu at (186.0, 91.0)
Other:
- board text added: "danman.eu cyusb3014-breakout v1.0"
